File: z80_computer.sch (KiCad schematic (older format))
At the start: 21 parts, among them J1 Screw_Terminal_01x02, J2 Bus_ISA_8bit, U1 74LS14, U2 MCP130, U3 LM117_TO3, U4 74LS32, U5 Z80CPU, Y1 Crystal

Commit message: Added ISA bus, broke some circuits into sub schematics.
Parts:
- removed U4: 74LS32, Package_DIP:DIP-14_W7.62mm, symbol 74xx:74LS32
Connections:
- net labels added: ~BOOT, ~D[0..7], ~INTACK, ~OPFETCH
- wire segments 164 -> 169

Commit message: Added demux for IO select
Parts:
- added R9: 10K, symbol Device:R_US
- added U8: 74138, symbol 74xx:74LS138
Connections:
- net labels added: DS0, DS1, DS2, DS3, DS4, DS5, DS6, DS7, DS[0..7]
- wire segments 169 -> 189

Commit message: Added some temporary footprints and messed with the oscillator layout
Parts:
- R9: footprint (none) -> Resistor_THT:R_Axial_DIN0207_L6.3mm_D2.5mm_P5.08mm_Vertical
- U8: footprint (none) -> Package_DIP:DIP-16_W7.62mm
Changed lines of the file:
@@
 F 0 "U8" H 1650 7200 50  0000 C CNN
 F 1 "74138" H 1650 7100 50  0000 C CNN
-F 2 "" H 1850 6650 50  0001 C CNN
+F 2 "Package_DIP:DIP-16_W7.62mm" H 1850 6650 50  0001 C CNN
 F 3 "http://www.ti.com/lit/gpn/sn74LS138" H 1850 6650 50  0001 C CNN
 	1    1850 6650
@@
 	1850 6050 1850 6000
 $Comp
-L power:+5V #PWR?
+L power:+5V #PWR0102
 U 1 1 5BD33ED3
 P 1850 6000
-F 0 "#PWR?" H 1850 5850 50  0001 C CNN
+F 0 "#PWR0102" H 1850 5850 50  0001 C CNN
 F 1 "+5V" H 1865 6173 50  0000 C CNN
 F 2 "" H 1850 6000 50  0001 C CNN
@@
 	1850 7350 1850 7400
 $Comp
-L power:GND #PWR?
+L power:GND #PWR0103
 U 1 1 5BDA3178
 P 1850 7400
-F 0 "#PWR?" H 1850 7150 50  0001 C CNN
+F 0 "#PWR0103" H 1850 7150 50  0001 C CNN
 F 1 "GND" H 1855 7227 50  0000 C CNN
 F 2 "" H 1850 7400 50  0001 C CNN
@@
 F 0 "R9" V 945 6850 50  0000 C CNN
 F 1 "10K" V 1036 6850 50  0000 C CNN
-F 2 "" V 1190 6840 50  0001 C CNN
+F 2 "Resistor_THT:R_Axial_DIN0207_L6.3mm_D2.5mm_P5.08mm_Vertical" V 1190 6840 50  0001 C CNN
 F 3 "~" H 1150 6850 50  0001 C CNN
 	1    1150 6850
@@
 	1000 7050 1250 7050
 $Comp
-L power:GND #PWR?
+L power:GND #PWR0104
 U 1 1 5BE4A11C
 P 750 6900
-F 0 "#PWR?" H 750 6650 50  0001 C CNN
+F 0 "#PWR0104" H 750 6650 50  0001 C CNN
 F 1 "GND" H 755 6727 50  0000 C CNN
 F 2 "" H 750 6900 50  0001 C CNN
@@
 	750  6850 1000 6850
 Wire Bus Line
-	5150 4650 5150 5350
+	9700 3700 9700 5200
+Wire Bus Line
+	5150 2950 5150 4450
+Wire Bus Line
+	2650 6450 2650 7150
 Wire Bus Line
 	9900 2300 9900 3000
 Wire Bus Line
-	2650 6450 2650 7150
-Wire Bus Line
-	5150 2950 5150 4450
-Wire Bus Line
-	9700 3700 9700 5200
+	5150 4650 5150 5350
 $EndSCHEMATC
